File: iso_40.kicad_pcb (KiCad board)
At the start: 2 copper layers, 238.1 x 78.6 mm, 96 parts, among them SW1 SW_Push, U1 ATmega32U4-AU, Y1 16MHz

Commit message: review
Parts:
- moved C6 0.79 mm to (128.6, 98.3)
Routing:
- net Net-(USB1-Pad6): track 0.00 -> 23.6 mm
- net row_3: track 201.3 -> 202.2 mm, vias 0 -> 2
- net col_11: track 168.9 -> 169.8 mm
- added copper zone on B.Cu, net GND
- added copper zone on F.Cu, net Net-(USB1-Pad6)
- added copper zone on F.Cu, net col_11
Other:
- board text added: "assembly iso 40"

Commit message: ISP header added
Parts:
- added J1: AVR-ISP-6, Connector_PinHeader_2.54mm:PinHeader_2x03_P2.54mm_Vertical, F.Cu at (127.0, 59.5)
- moved D13 7.33 mm to (42.1, 49.2)
Connections:
- net Net-(R1-Pad2) renamed reset
- net col_07 renamed SCLK
- net col_08 renamed MOSI
- net col_09 renamed MISO
- R2 pad 1: Net-(R2-Pad1) -> D+
- R2 pad 2: D+ -> pre_D+
- R3 pad 1: Net-(R3-Pad1) -> D-
- R3 pad 2: D- -> pre_D-
- U1 pad 3: Net-(R3-Pad1) -> D-
- U1 pad 4: Net-(R2-Pad1) -> D+
- USB1 pad 3: D+ -> pre_D+
- USB1 pad 4: D- -> pre_D-
Routing:
- net Net-(R3-Pad1): track 115.2 -> 0.00 mm, vias 4 -> 0
- net Net-(R2-Pad1): track 111.7 -> 0.00 mm, vias 4 -> 0
- net D-: track 7.41 -> 106.7 mm
- net D+: track 8.06 -> 106.7 mm
- net +5V: track 246.2 -> 291.7 mm, vias 9 -> 12
- net GND: track 236.4 -> 261.5 mm, vias 3 -> 6
- net MISO: track 150.6 -> 175.2 mm
- net SCLK: track 105.4 -> 125.1 mm, vias 3 -> 4
- net MOSI: track 123.3 -> 141.1 mm, vias 3 -> 5
- net reset: track 132.8 -> 147.6 mm, vias 6 -> 7
- net Net-(R4-Pad2): track 129.2 -> 115.3 mm
- net pre_D-: track 0.00 -> 8.22 mm
- net pre_D+: track 0.00 -> 8.06 mm
- net Net-(D13-Pad2): track 9.29 -> 3.01 mm
- net col_02: track 98.6 -> 100.6 mm
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- removed copper zone on F.Cu, net col_11

Commit message: pcb changes, etc
Parts:
- removed USB1: Molex-0548190589, random-keyboard-parts:Molex-0548190589
- added J2: USB_C_Receptacle_USB2.0_16P, Connector_USB:USB_C_Receptacle_GCT_USB4110, B.Cu at (44.8, 23.1)
- J1: footprint Connector_PinHeader_2.54mm:PinHeader_2x03_P2.54mm_Vertical -> Connector_PinHeader_2.54mm:PinHeader_2x03_P2.54mm_Vertical_SMD
- MX29: moved to B.Cu
- moved J1 57.5 mm to (175.4, 90.5), turned to 90 degrees
- moved D1 0.06 mm to (34.9, 38.1)
- turned MX29 to 180 degrees
Connections:
- U1 pad 1: Net-(U1-Pad1) -> unconnected-(U1-PE6-Pad1)
- U1 pad 26: Net-(U1-Pad26) -> unconnected-(U1-PD6-Pad26)
- U1 pad 27: Net-(U1-Pad27) -> unconnected-(U1-PD7-Pad27)
- U1 pad 28: Net-(U1-Pad28) -> unconnected-(U1-PB4-Pad28)
- U1 pad 29: Net-(U1-Pad29) -> unconnected-(U1-PB5-Pad29)
- U1 pad 30: Net-(U1-Pad30) -> unconnected-(U1-PB6-Pad30)
- U1 pad 31: Net-(U1-Pad31) -> unconnected-(U1-PC6-Pad31)
- U1 pad 32: Net-(U1-Pad32) -> unconnected-(U1-PC7-Pad32)
- U1 pad 36: Net-(U1-Pad36) -> unconnected-(U1-PF7-Pad36)
- U1 pad 42: Net-(U1-Pad42) -> unconnected-(U1-AREF-Pad42)
Routing:
- net reset: track 147.6 -> 200.7 mm, vias 7 -> 10
- net Net-(USB1-Pad6): track 23.6 -> 0.00 mm
- net MISO: track 175.2 -> 195.1 mm
- net GND: track 261.5 -> 276.7 mm, vias 6 -> 3
- net VCC: track 7.26 -> 21.2 mm, vias 0 -> 2
- net row_1: track 245.0 -> 257.2 mm, vias 2 -> 4
- net col_05: track 68.1 -> 78.0 mm
- net pre_D+: track 8.06 -> 16.1 mm
- net pre_D-: track 8.22 -> 14.2 mm
- net Net-(D29-A): track 8.05 -> 13.8 mm
- net SCLK: track 125.1 -> 130.6 mm
- net Net-(U1-~{HWB}/PE2): track 115.3 -> 120.0 mm, vias 6 -> 4
- net row_3: track 202.2 -> 206.8 mm
- net MOSI: track 141.1 -> 136.5 mm, vias 5 -> 3
- net col_02: track 100.6 -> 98.6 mm
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- added copper zone on F.Cu, net GND
- removed copper zone on F.Cu, net Net-(USB1-Pad6)
Other:
- board size 238.1 x 78.6 mm -> 238.1 x 83.3 mm
- net class Default removed
- net class Power removed
- board text added: "TENDER MENDING SENDER"
- board text added: "tender_mending_sender"
- board text removed: "assembly iso 40"
